File: firstTraining.sch (KiCad schematic (older format))
At the start: 17 parts, among them T1 Transformer_1P_SS, U1 TA48M05F, U2 TA48033S

Commit message: フットプリントとネットリスト更新
Parts:
- C1: footprint Capacitor_THT:CP_Radial_D10.0mm_P5.00mm -> Capacitor_THT:CP_Radial_D18.0mm_P7.50mm
- C3, C4: footprint Capacitor_THT:CP_Radial_D10.0mm_P5.00mm -> Capacitor_THT:CP_Radial_D5.0mm_P2.00mm
Changed lines of the file:
@@
 F 0 "C1" H 4865 1696 50  0000 L CNN
 F 1 "CP1" H 4865 1605 50  0000 L CNN
-F 2 "Capacitor_THT:CP_Radial_D10.0mm_P5.00mm" H 4750 1650 50  0001 C CNN
+F 2 "Capacitor_THT:CP_Radial_D18.0mm_P7.50mm" H 4750 1650 50  0001 C CNN
 F 3 "~" H 4750 1650 50  0001 C CNN
 	1    4750 1650
@@
 F 0 "C3" H 7315 1696 50  0000 L CNN
 F 1 "CP1" H 7315 1605 50  0000 L CNN
-F 2 "Capacitor_THT:CP_Radial_D10.0mm_P5.00mm" H 7200 1650 50  0001 C CNN
+F 2 "Capacitor_THT:CP_Radial_D5.0mm_P2.00mm" H 7200 1650 50  0001 C CNN
 F 3 "~" H 7200 1650 50  0001 C CNN
 	1    7200 1650
@@
 F 0 "C4" H 7315 2546 50  0000 L CNN
 F 1 "CP1" H 7315 2455 50  0000 L CNN
-F 2 "Capacitor_THT:CP_Radial_D10.0mm_P5.00mm" H 7200 2500 50  0001 C CNN
+F 2 "Capacitor_THT:CP_Radial_D5.0mm_P2.00mm" H 7200 2500 50  0001 C CNN
 F 3 "~" H 7200 2500 50  0001 C CNN
 	1    7200 2500

Commit message: フットプリント更新した
Parts:
- U1, U2: footprint Connector_PinHeader_2.54mm:PinHeader_1x03_P2.54mm_Vertical -> newLib:TOSHIBA_DIP_Regulators
Changed lines of the file:
@@
 F 0 "U2" H 6575 2875 50  0000 C CNN
 F 1 "TA48033S" H 6575 2784 50  0000 C CNN
-F 2 "Connector_PinHeader_2.54mm:PinHeader_1x03_P2.54mm_Vertical" H 6550 2500 50  0001 C CNN
+F 2 "newLib:TOSHIBA_DIP_Regulators" H 6550 2500 50  0001 C CNN
 F 3 "" H 6550 2500 50  0001 C CNN
 	1    6550 2500
@@
 F 0 "U1" H 6500 1865 50  0000 C CNN
 F 1 "TA48M05F" H 6500 1774 50  0000 C CNN
-F 2 "Connector_PinHeader_2.54mm:PinHeader_1x03_P2.54mm_Vertical" H 6450 1550 50  0001 C CNN
+F 2 "newLib:TOSHIBA_DIP_Regulators" H 6450 1550 50  0001 C CNN
 F 3 "" H 6450 1550 50  0001 C CNN
 	1    6450 1550
